File: Hardware/sequencer.sch (KiCad schematic (older format))
At the start: 100 parts, among them IC1 74HC165N, IC2 74HC165N, IC3 74HC165N, IC4 74HC165N, J1 SJ-3523-SMT-TR, U1 Teensy3.6

Commit message: PCB rev 1.2
Connections:
- net Audio1: now also J1.3; no longer J1.2
- net Audio2: now also J1.2; no longer J1.3
Changed lines of the file:
@@
 	1    0    0    -1
 $EndComp
-Text Label 11850 16600 0    60   ~ 0
+Text Label 11850 16450 0    60   ~ 0
 Audio1
 Text Label 13050 16200 2    60   ~ 0
 Audio1
-Text Label 11850 16450 0    60   ~ 0
+Text Label 11850 16600 0    60   ~ 0
 Audio2
 Text Label 13050 16450 2    60   ~ 0

Commit message: rev 1.3 pcb - Pots rotated by 180 degrees - Added circuit for trigger input
Parts:
- added D31: 1N4148, Diodes_THT:D_DO-35_SOD27_P2.54mm_Vertical_AnodeUp, symbol 1N4148
- added J2: SJ-3523-SMT-TR, SJ-3523-SMT-TR:CUI_SJ-3523-SMT-TR, symbol SJ-3523-SMT-TR
- added Q1: 2N3904, TO_SOT_Packages_THT:TO-92_Inline_Wide, symbol 2N3904
- added R31, R32: 10k, Resistors_SMD:R_1206_HandSoldering, symbol R-US_0204_2V
Connections:
- net GND: now also D31.2 (A), J2.1, Q1.1 (E)
- net VCC: now also R32.2
- net Trigger-Input: now reaches U1.30 (33_A14_CAN1TX_scl0)
- net Trigger-Input: now also Q1.3 (C), R32.1
- new net: J2.2, R31.1
- new net: D31.1 (K), Q1.2 (B), R31.2
Changed lines of the file:
@@
 LIBS:SJ-3523-SMT-TR
 LIBS:device
+LIBS:diode
+LIBS:Transistor_BJT
 LIBS:sequencer-cache
 EELAYER 25 0
@@
 	9150 10650 9650 10650
 Wire Wire Line
-	9650 10350 9150 10350
-Wire Wire Line
-	9650 10050 9150 10050
-Wire Wire Line
-	9650 9750 9150 9750
-Wire Wire Line
-	9650 9450 9150 9450
+	9150 10350 9650 10350
+Wire Wire Line
+	9150 10050 9650 10050
+Wire Wire Line
+	9150 9750 9650 9750
+Wire Wire Line
+	9150 9450 9650 9450
 Wire Wire Line
 	9650 9150 9150 9150
@@
 	4550 11000 5050 11000
 Wire Wire Line
-	5050 10700 4550 10700
-Wire Wire Line
-	5050 10400 4550 10400
-Wire Wire Line
-	5050 10100 4550 10100
-Wire Wire Line
-	5050 9800 4550 9800
-Wire Wire Line
-	5050 9500 4550 9500
+	4550 10700 5050 10700
+Wire Wire Line
+	4550 10400 5050 10400
+Wire Wire Line
+	4550 10100 5050 10100
+Wire Wire Line
+	4550 9800 5050 9800
+Wire Wire Line
+	4550 9500 5050 9500
 Wire Wire Line
 	5050 9200 4550 9200
@@
 	1    13150 16450
 	0    1    1    0
-$EndComp
-$Comp
-L Teensy3.6 U1
-U 1 1 5BACEF6D
-P 14900 14700
-F 0 "U1" H 14900 17000 60  0000 C CNN
-F 1 "Teensy3.6" H 14900 12400 60  0000 C CNN
-F 2 "modules:Teensy35_36_simple" H 14900 14700 60  0001 C CNN
-F 3 "" H 14900 14700 60  0000 C CNN
-	1    14900 14700
-	1    0    0    -1
 $EndComp
 Text Label 11850 16450 0    60   ~ 0
@@
 	1    0    0    -1
 $EndComp
+$Comp
+L SJ-3523-SMT-TR J2
+U 1 1 5C9CE2B4
+P 18050 12800
+F 0 "J2" H 17849 13026 50  0000 L BNN
+F 1 "SJ-3523-SMT-TR" H 17849 12499 50  0000 L BNN
+F 2 "SJ-3523-SMT-TR:CUI_SJ-3523-SMT-TR" H 18050 12800 50  0001 L BNN
+F 3 "Manufacturer recommendations" H 18050 12800 50  0001 L BNN
+F 4 "CUI Inc" H 18050 12800 50  0001 L BNN "Feld4"
+	1    18050 12800
+	1    0    0    -1
+$EndComp
+$Comp
+L R-US_0204_2V R32
+U 1 1 5C9CE7F6
+P 19500 12450
+F 0 "R32" H 19350 12508 70  0000 L BNN
+F 1 "10k" H 19350 12320 70  0000 L BNN
+F 2 "Resistors_SMD:R_1206_HandSoldering" H 19490 12240 65  0001 L TNN
+F 3 "" H 19500 12450 60  0001 C CNN
+	1    19500 12450
+	0    -1   -1   0
+$EndComp
+$Comp
+L R-US_0204_2V R31
+U 1 1 5C9CEAEB
+P 18800 12900
+F 0 "R31" H 18650 12958 70  0000 L BNN
+F 1 "10k" H 18650 12770 70  0000 L BNN
+F 2 "Resistors_SMD:R_1206_HandSoldering" H 18790 12690 65  0001 L TNN
+F 3 "" H 18800 12900 60  0001 C CNN
+	1    18800 12900
+	1    0    0    -1
+$EndComp
+$Comp
+L 2N3904 Q1
+U 1 1 5C9CF599
+P 19400 12900
+F 0 "Q1" H 19600 12975 50  0000 L CNN
+F 1 "2N3904" H 19600 12900 50  0000 L CNN
+F 2 "TO_SOT_Packages_THT:TO-92_Inline_Wide" H 19600 12825 50  0001 L CIN
+F 3 "" H 19400 12900 50  0001 L CNN
+	1    19400 12900
+	1    0    0    -1
+$EndComp
+$Comp
+L 1N4148 D31
+U 1 1 5C9CFA2D
+P 19350 13200
+F 0 "D31" H 19350 13300 50  0000 C CNN
+F 1 "1N4148" H 19350 13100 50  0000 C CNN
+F 2 "Diodes_THT:D_DO-35_SOD27_P2.54mm_Vertical_AnodeUp" H 19350 13025 50  0001 C CNN
+F 3 "" H 19350 13200 50  0001 C CNN
+	1    19350 13200
+	1    0    0    -1
+$EndComp
+$Comp
+L VCC #SUPPLY036
+U 1 1 5C9CFE9E
+P 19500 12200
+F 0 "#SUPPLY036" H 19500 12200 45  0001 L BNN
+F 1 "VCC" H 19460 12340 45  0000 L BNN
+F 2 "" H 19500 12200 60  0001 C CNN
+F 3 "" H 19500 12200 60  0001 C CNN
+	1    19500 12200
+	1    0    0    -1
+$EndComp
+$Comp
+L GND #GND037
+U 1 1 5C9CFFF0
+P 19500 13600
+F 0 "#GND037" H 19400 13500 70  0001 L BNN
+F 1 "GND" H 19400 13500 70  0000 L BNN
+F 2 "" H 19500 13600 60  0001 C CNN
+F 3 "" H 19500 13600 60  0001 C CNN
+	1    19500 13600
+	1    0    0    -1
+$EndComp
+Wire Wire Line
+	19500 12650 19500 12700
+Wire Wire Line
+	19000 12900 19200 12900
+Wire Wire Line
+	19500 13100 19500 13500
+Connection ~ 19500 13200
+Wire Wire Line
+	19200 12900 19200 13200
+Connection ~ 19200 12900
+$Comp
+L GND #GND038
+U 1 1 5C9D2173
+P 18350 12450
+F 0 "#GND038" H 18250 12350 70  0001 L BNN
+F 1 "GND" H 18250 12350 70  0000 L BNN
+F 2 "" H 18350 12450 60  0001 C CNN
+F 3 "" H 18350 12450 60  0001 C CNN
+	1    18350 12450
+	-1   0    0    1
+$EndComp
+Wire Wire Line
+	18350 12700 18350 12550
+Text Label 13900 15500 2    60   ~ 0
+Trigger-Input
+Text Label 19900 12700 0    60   ~ 0
+Trigger-Input
+Wire Wire Line
+	19500 12700 19900 12700
+Connection ~ 19500 12700
+Wire Wire Line
+	19500 12200 19500 12250
+Wire Wire Line
+	18350 12900 18600 12900
+$Comp
+L Teensy3.6 U1
+U 1 1 5BACEF6D
+P 14900 14700
+F 0 "U1" H 14900 17000 60  0000 C CNN
+F 1 "Teensy3.6" H 14900 12400 60  0000 C CNN
+F 2 "modules:Teensy35_36_simple" H 14900 14700 60  0001 C CNN
+F 3 "" H 14900 14700 60  0000 C CNN
+	1    14900 14700
+	1    0    0    -1
+$EndComp

Commit message: Hardware Rev 1.4: Function buttons and track buttons now use SMD Resistors, so that there is space on the PCB for text labels for each function button
Parts:
- R17, R18, R19, R20, R21, R22, R23, R24, R25, R26, R27, R28, R29, R30: footprint modules:R_Axial_DIN0411_L9.9mm_D3.6mm_P12.70mm_Horizontal_noSilkscreen -> Resistors_SMD:R_1206_HandSoldering
Changed lines of the file:
@@
 F 0 "R25" H 10300 9208 70  0000 L BNN
 F 1 "270" H 10300 9020 70  0000 L BNN
-F 2 "modules:R_Axial_DIN0411_L9.9mm_D3.6mm_P12.70mm_Horizontal_noSilkscreen" H 10440 8940 65  0001 L TNN
+F 2 "Resistors_SMD:R_1206_HandSoldering" H 10440 8940 65  0001 L TNN
 F 3 "" H 10450 9150 60  0001 C CNN
 	1    10450 9150
@@
 F 0 "R26" H 10300 9508 70  0000 L BNN
 F 1 "270" H 10300 9320 70  0000 L BNN
-F 2 "modules:R_Axial_DIN0411_L9.9mm_D3.6mm_P12.70mm_Horizontal_noSilkscreen" H 10440 9240 65  0001 L TNN
+F 2 "Resistors_SMD:R_1206_HandSoldering" H 10440 9240 65  0001 L TNN
 F 3 "" H 10450 9450 60  0001 C CNN
 	1    10450 9450
@@
 F 0 "R27" H 10300 9808 70  0000 L BNN
 F 1 "270" H 10300 9620 70  0000 L BNN
-F 2 "modules:R_Axial_DIN0411_L9.9mm_D3.6mm_P12.70mm_Horizontal_noSilkscreen" H 10440 9540 65  0001 L TNN
+F 2 "Resistors_SMD:R_1206_HandSoldering" H 10440 9540 65  0001 L TNN
 F 3 "" H 10450 9750 60  0001 C CNN
 	1    10450 9750
@@
 F 0 "R28" H 10300 10108 70  0000 L BNN
 F 1 "270" H 10300 9920 70  0000 L BNN
-F 2 "modules:R_Axial_DIN0411_L9.9mm_D3.6mm_P12.70mm_Horizontal_noSilkscreen" H 10440 9840 65  0001 L TNN
+F 2 "Resistors_SMD:R_1206_HandSoldering" H 10440 9840 65  0001 L TNN
 F 3 "" H 10450 10050 60  0001 C CNN
 	1    10450 10050
@@
 F 0 "R29" H 10300 10408 70  0000 L BNN
 F 1 "270" H 10300 10220 70  0000 L BNN
-F 2 "modules:R_Axial_DIN0411_L9.9mm_D3.6mm_P12.70mm_Horizontal_noSilkscreen" H 10440 10140 65  0001 L TNN
+F 2 "Resistors_SMD:R_1206_HandSoldering" H 10440 10140 65  0001 L TNN
 F 3 "" H 10450 10350 60  0001 C CNN
 	1    10450 10350
@@
 F 0 "R30" H 10300 10708 70  0000 L BNN
 F 1 "270" H 10300 10520 70  0000 L BNN
-F 2 "modules:R_Axial_DIN0411_L9.9mm_D3.6mm_P12.70mm_Horizontal_noSilkscreen" H 10440 10440 65  0001 L TNN
+F 2 "Resistors_SMD:R_1206_HandSoldering" H 10440 10440 65  0001 L TNN
 F 3 "" H 10450 10650 60  0001 C CNN
 	1    10450 10650
@@
 F 0 "R17" H 5700 5558 70  0000 L BNN
 F 1 "270" H 5700 5370 70  0000 L BNN
-F 2 "modules:R_Axial_DIN0411_L9.9mm_D3.6mm_P12.70mm_Horizontal_noSilkscreen" H 5840 5290 65  0001 L TNN
+F 2 "Resistors_SMD:R_1206_HandSoldering" H 5840 5290 65  0001 L TNN
 F 3 "" H 5850 5500 60  0001 C CNN
 	1    5850 5500
@@
 F 0 "R18" H 5700 5858 70  0000 L BNN
 F 1 "270" H 5700 5670 70  0000 L BNN
-F 2 "modules:R_Axial_DIN0411_L9.9mm_D3.6mm_P12.70mm_Horizontal_noSilkscreen" H 5840 5590 65  0001 L TNN
+F 2 "Resistors_SMD:R_1206_HandSoldering" H 5840 5590 65  0001 L TNN
 F 3 "" H 5850 5800 60  0001 C CNN
 	1    5850 5800
@@
 F 0 "R19" H 5700 6158 70  0000 L BNN
 F 1 "270" H 5700 5970 70  0000 L BNN
-F 2 "modules:R_Axial_DIN0411_L9.9mm_D3.6mm_P12.70mm_Horizontal_noSilkscreen" H 5840 5890 65  0001 L TNN
+F 2 "Resistors_SMD:R_1206_HandSoldering" H 5840 5890 65  0001 L TNN
 F 3 "" H 5850 6100 60  0001 C CNN
 	1    5850 6100
@@
 F 0 "R20" H 5700 6458 70  0000 L BNN
 F 1 "270" H 5700 6270 70  0000 L BNN
-F 2 "modules:R_Axial_DIN0411_L9.9mm_D3.6mm_P12.70mm_Horizontal_noSilkscreen" H 5840 6190 65  0001 L TNN
+F 2 "Resistors_SMD:R_1206_HandSoldering" H 5840 6190 65  0001 L TNN
 F 3 "" H 5850 6400 60  0001 C CNN
 	1    5850 6400
@@
 F 0 "R21" H 5700 6758 70  0000 L BNN
 F 1 "270" H 5700 6570 70  0000 L BNN
-F 2 "modules:R_Axial_DIN0411_L9.9mm_D3.6mm_P12.70mm_Horizontal_noSilkscreen" H 5840 6490 65  0001 L TNN
+F 2 "Resistors_SMD:R_1206_HandSoldering" H 5840 6490 65  0001 L TNN
 F 3 "" H 5850 6700 60  0001 C CNN
 	1    5850 6700
@@
 F 0 "R22" H 5700 7058 70  0000 L BNN
 F 1 "270" H 5700 6870 70  0000 L BNN
-F 2 "modules:R_Axial_DIN0411_L9.9mm_D3.6mm_P12.70mm_Horizontal_noSilkscreen" H 5840 6790 65  0001 L TNN
+F 2 "Resistors_SMD:R_1206_HandSoldering" H 5840 6790 65  0001 L TNN
 F 3 "" H 5850 7000 60  0001 C CNN
 	1    5850 7000
@@
 F 0 "R23" H 5700 7358 70  0000 L BNN
 F 1 "270" H 5700 7170 70  0000 L BNN
-F 2 "modules:R_Axial_DIN0411_L9.9mm_D3.6mm_P12.70mm_Horizontal_noSilkscreen" H 5840 7090 65  0001 L TNN
+F 2 "Resistors_SMD:R_1206_HandSoldering" H 5840 7090 65  0001 L TNN
 F 3 "" H 5850 7300 60  0001 C CNN
 	1    5850 7300
@@
 F 0 "R24" H 5700 7658 70  0000 L BNN
 F 1 "270" H 5700 7470 70  0000 L BNN
-F 2 "modules:R_Axial_DIN0411_L9.9mm_D3.6mm_P12.70mm_Horizontal_noSilkscreen" H 5840 7390 65  0001 L TNN
+F 2 "Resistors_SMD:R_1206_HandSoldering" H 5840 7390 65  0001 L TNN
 F 3 "" H 5850 7600 60  0001 C CNN
 	1    5850 7600
